File: examples/sandwich-example/sandwich-example.kicad_pcb (KiCad board)
At the start: 4 copper layers, 100 x 80 mm, 2 parts, among them U1 LM555xM, U2 LM555xM

Commit message: Updated basic example to v6 standard directory format
Other:
- net class Default removed
